Commit message: Add: codes for backflip and sideflip trajectory optimization

File: robots/p73/urdf/p73.urdf (robot description, URDF)
Before this commit: robot P73, 33 links, 32 joints
Joints:
- joint L_AnklePitch_Joint: limit lower=-3.14 upper=3.14 effort=300.0 velocity=10.0 -> lower=-3.14 upper=3.14 effort=500.0 velocity=10.0
- joint L_AnkleRoll_Joint: limit lower=-3.14 upper=3.14 effort=300.0 velocity=10.0 -> lower=-3.14 upper=3.14 effort=500.0 velocity=10.0
- joint L_Elbow_Joint: limit lower=-3.14 upper=3.14 effort=300.0 velocity=10.0 -> lower=-3.14 upper=3.14 effort=500.0 velocity=10.0
- joint L_HipPitch_Joint: limit lower=-3.14 upper=3.14 effort=300.0 velocity=10.0 -> lower=-3.14 upper=3.14 effort=500.0 velocity=10.0
- joint L_HipRoll_Joint: limit lower=-3.14 upper=3.14 effort=300.0 velocity=10.0 -> lower=-3.14 upper=3.14 effort=500.0 velocity=10.0
- joint L_HipYaw_Joint: limit lower=-3.14 upper=3.14 effort=300.0 velocity=10.0 -> lower=-3.14 upper=3.14 effort=500.0 velocity=10.0
- joint L_Knee_Joint: limit lower=-3.14 upper=3.14 effort=300.0 velocity=10.0 -> lower=-3.14 upper=3.14 effort=500.0 velocity=10.0
- joint L_ShoulderPitch_Joint: limit lower=-3.14 upper=3.14 effort=300.0 velocity=10.0 -> lower=-3.14 upper=3.14 effort=500.0 velocity=10.0
- joint L_ShoulderRoll_Joint: limit lower=-3.14 upper=3.14 effort=300.0 velocity=10.0 -> lower=-3.14 upper=3.14 effort=500.0 velocity=10.0
- joint L_ShoulderYaw_Joint: limit lower=-3.14 upper=3.14 effort=300.0 velocity=10.0 -> lower=-3.14 upper=3.14 effort=500.0 velocity=10.0
- joint L_WristPitch_Joint: limit lower=-3.14 upper=3.14 effort=300.0 velocity=10.0 -> lower=-3.14 upper=3.14 effort=500.0 velocity=10.0
- joint L_WristRoll_Joint: limit lower=-3.14 upper=3.14 effort=300.0 velocity=10.0 -> lower=-3.14 upper=3.14 effort=500.0 velocity=10.0
- joint L_WristYaw_Joint: limit lower=-3.14 upper=3.14 effort=300.0 velocity=10.0 -> lower=-3.14 upper=3.14 effort=500.0 velocity=10.0
- joint NeckPitch_Joint: limit lower=-3.14 upper=3.14 effort=300.0 velocity=10.0 -> lower=-3.14 upper=3.14 effort=500.0 velocity=10.0
- joint NeckRoll_Joint: limit lower=-3.14 upper=3.14 effort=300.0 velocity=10.0 -> lower=-3.14 upper=3.14 effort=500.0 velocity=10.0
- joint NeckYaw_Joint: limit lower=-3.14 upper=3.14 effort=300.0 velocity=10.0 -> lower=-3.14 upper=3.14 effort=500.0 velocity=10.0
- joint R_AnklePitch_Joint: limit lower=-3.14 upper=3.14 effort=300.0 velocity=10.0 -> lower=-3.14 upper=3.14 effort=500.0 velocity=10.0
- joint R_AnkleRoll_Joint: limit lower=-3.14 upper=3.14 effort=300.0 velocity=10.0 -> lower=-3.14 upper=3.14 effort=500.0 velocity=10.0
- joint R_Elbow_Joint: limit lower=-3.14 upper=3.14 effort=300.0 velocity=10.0 -> lower=-3.14 upper=3.14 effort=500.0 velocity=10.0
- joint R_HipPitch_Joint: limit lower=-3.14 upper=3.14 effort=300.0 velocity=10.0 -> lower=-3.14 upper=3.14 effort=500.0 velocity=10.0
- joint R_HipRoll_Joint: limit lower=-3.14 upper=3.14 effort=300.0 velocity=10.0 -> lower=-3.14 upper=3.14 effort=500.0 velocity=10.0
- joint R_HipYaw_Joint: limit lower=-3.14 upper=3.14 effort=300.0 velocity=10.0 -> lower=-3.14 upper=3.14 effort=500.0 velocity=10.0
- joint R_Knee_Joint: limit lower=-3.14 upper=3.14 effort=300.0 velocity=10.0 -> lower=-3.14 upper=3.14 effort=500.0 velocity=10.0
- joint R_ShoulderPitch_Joint: limit lower=-3.14 upper=3.14 effort=300.0 velocity=10.0 -> lower=-3.14 upper=3.14 effort=500.0 velocity=10.0
- joint R_ShoulderRoll_Joint: limit lower=-3.14 upper=3.14 effort=300.0 velocity=10.0 -> lower=-3.14 upper=3.14 effort=500.0 velocity=10.0
- joint R_ShoulderYaw_Joint: limit lower=-3.14 upper=3.14 effort=300.0 velocity=10.0 -> lower=-3.14 upper=3.14 effort=500.0 velocity=10.0
- joint R_WristPitch_Joint: limit lower=-3.14 upper=3.14 effort=300.0 velocity=10.0 -> lower=-3.14 upper=3.14 effort=500.0 velocity=10.0
- joint R_WristRoll_Joint: limit lower=-3.14 upper=3.14 effort=300.0 velocity=10.0 -> lower=-3.14 upper=3.14 effort=500.0 velocity=10.0
- joint R_WristYaw_Joint: limit lower=-3.14 upper=3.14 effort=300.0 velocity=10.0 -> lower=-3.14 upper=3.14 effort=500.0 velocity=10.0
- joint WaistPitch_Joint: limit lower=-3.14 upper=3.14 effort=300.0 velocity=10.0 -> lower=-3.14 upper=3.14 effort=500.0 velocity=10.0
- joint WaistRoll_Joint: limit lower=-3.14 upper=3.14 effort=300.0 velocity=10.0 -> lower=-3.14 upper=3.14 effort=500.0 velocity=10.0
- joint WaistYaw_Joint: limit lower=-3.14 upper=3.14 effort=300.0 velocity=10.0 -> lower=-3.14 upper=3.14 effort=500.0 velocity=10.0

Commit message: p73 walker version

File: robots/p73/urdf/p73.urdf (robot description, URDF)
Before this commit: robot P73, 33 links, 32 joints
Links:
- removed link Head_1
- removed link L_AnkleRoll_Link_1
- removed link L_Elbow_Link_1
- removed link L_Foot_Link_1
- removed link L_HipPitch_Link_1
- removed link L_HipRoll_Link_1
- removed link L_Knee_Link_1
- removed link L_ShoulderPitch_Link_1
- removed link L_ShoulderRoll_Link_1
- removed link L_Thigh_Link_1
- removed link L_UpperArm_Link_1
- removed link L_WristPitch_Link_1
- removed link L_WristRoll_Link_1
- removed link L_WristYaw_Link_1
- removed link NeckPitch_Link_1
- removed link NeckRoll_Link_1
- removed link R_AnkleRoll_Link_1
- removed link R_Elbow_Link_1
- removed link R_Foot_Link_1
- removed link R_HipPitch_Link_1
- removed link R_HipRoll_Link_1
- removed link R_Knee_Link_1
- removed link R_ShoulderPitch_Link_1
- removed link R_ShoulderRoll_Link_1
- removed link R_Thigh_Link_1
- removed link R_UpperArm_Link_1
- removed link R_WristPitch_Link_1
- removed link R_WristRoll_Link_1
- removed link R_WristYaw_Link_1
- removed link Torso_1
- removed link WaistRoll_Link_1
- removed link WaistYaw_Link_1
- added link L_AnkleRoll_Link, mass 0.16126824126437989; collision mesh filename=../meshes/L_AnkleRoll_Link.stl scale=0.001 0.001 0.001; visual mesh filename=../meshes/L_AnkleRoll_Link.stl scale=0.001 0.001 0.001
- added link L_Foot_Link, mass 2.3290372118414675; collision box size=0.06 0.1 0.02; collision box size=0.2 0.1 0.02
- added link L_HipPitch_Link, mass 6.857435533216696; collision box size=0.2 0.11 0.26; visual mesh filename=../meshes/L_HipPitch_Link.stl scale=0.001 0.001 0.001
- added link L_HipRoll_Link, mass 1.2702673584378412; collision mesh filename=../meshes/L_HipRoll_Link.stl scale=0.001 0.001 0.001; visual mesh filename=../meshes/L_HipRoll_Link.stl scale=0.001 0.001 0.001
- added link L_Knee_Link, mass 8.18144928150599; collision box size=0.09 0.08 0.16; collision box size=0.12 0.12 0.24
- added link L_Thigh_Link, mass 4.903279724820187; collision box size=0.2 0.14 0.16; visual mesh filename=../meshes/L_Thigh_Link.stl scale=0.001 0.001 0.001
- added link R_AnkleRoll_Link, mass 0.16126824126437989; collision mesh filename=../meshes/R_AnkleRoll_Link.stl scale=0.001 0.001 0.001; visual mesh filename=../meshes/R_AnkleRoll_Link.stl scale=0.001 0.001 0.001
- added link R_Foot_Link, mass 2.3290370755141745; collision box size=0.06 0.1 0.02; collision box size=0.2 0.1 0.02
- added link R_HipPitch_Link, mass 6.857456505757582; collision box size=0.2 0.11 0.26; visual mesh filename=../meshes/R_HipPitch_Link.stl scale=0.001 0.001 0.001
- added link R_HipRoll_Link, mass 1.1787850921827068; collision mesh filename=../meshes/R_HipRoll_Link.stl scale=0.001 0.001 0.001; visual mesh filename=../meshes/R_HipRoll_Link.stl scale=0.001 0.001 0.001
- added link R_Knee_Link, mass 7.966815282700452; collision box size=0.09 0.08 0.16; collision box size=0.12 0.12 0.24
- added link R_Thigh_Link, mass 4.995693817886645; collision box size=0.2 0.14 0.16; visual mesh filename=../meshes/R_Thigh_Link.stl scale=0.001 0.001 0.001
- added link WaistYaw_Link, mass 7.605387605261044; collision box size=0.26 0.3 0.4; collision cylinder length=0.04 radius=0.065
- link base_link: mass 7.490079182026984 -> 5.475055271656153; geometry collision cylinder length=0.21 radius=0.065; visual mesh filename=../meshes/base_link.stl scale=0.001 0.001 0.001
Joints:
- removed joint L_Elbow_Joint
- removed joint L_ShoulderPitch_Joint
- removed joint L_ShoulderRoll_Joint
- removed joint L_ShoulderYaw_Joint
- removed joint L_WristPitch_Joint
- removed joint L_WristRoll_Joint
- removed joint L_WristYaw_Joint
- removed joint NeckPitch_Joint
- removed joint NeckRoll_Joint
- removed joint NeckYaw_Joint
- removed joint R_Elbow_Joint
- removed joint R_ShoulderPitch_Joint
- removed joint R_ShoulderRoll_Joint
- removed joint R_ShoulderYaw_Joint
- removed joint R_WristPitch_Joint
- removed joint R_WristRoll_Joint
- removed joint R_WristYaw_Joint
- removed joint WaistPitch_Joint
- removed joint WaistRoll_Joint
- joint L_AnklePitch_Joint: axis -0.0 1.0 -0.0 -> 0.0 1.0 -0.0; child L_AnkleRoll_Link_1 -> L_AnkleRoll_Link; limit lower=-3.14 upper=3.14 effort=500.0 velocity=10.0 -> lower=-1.05 upper=0.7 effort=95 velocity=10; origin xyz=0.043642 -0.0415 -0.415855 rpy=0 0 0 -> xyz=0.043642 -0.0025 -0.415855 rpy=0 0 0; parent L_Knee_Link_1 -> L_Knee_Link
- joint L_AnkleRoll_Joint: child L_Foot_Link_1 -> L_Foot_Link; limit lower=-3.14 upper=3.14 effort=500.0 velocity=10.0 -> lower=-0.42 upper=0.42 effort=95 velocity=10; parent L_AnkleRoll_Link_1 -> L_AnkleRoll_Link
- joint L_HipPitch_Joint: axis 0.0 -1.0 -0.0 -> -0.0 -1.0 -0.0; child L_HipPitch_Link_1 -> L_HipPitch_Link; limit lower=-3.14 upper=3.14 effort=500.0 velocity=10.0 -> lower=-1.57 upper=2.09 effort=220.0 velocity=10; origin xyz=0.0075 0.071 0.0 rpy=0 0 0 -> xyz=0.0155 0.0805 0.0 rpy=0 0 0; parent L_HipRoll_Link_1 -> L_HipRoll_Link
- joint L_HipRoll_Joint: axis 1.0 -0.0 0.0 -> 1.0 0.0 0.0; child L_HipRoll_Link_1 -> L_HipRoll_Link; limit lower=-3.14 upper=3.14 effort=500.0 velocity=10.0 -> lower=-0.58 upper=0.3 effort=352.0 velocity=10; origin xyz=-0.0075 0.0 0.0 rpy=0 0 0 -> xyz=-0.0155 0.0 0.0 rpy=0 0 0
- joint L_HipYaw_Joint: axis 0.0 0.0 -1.0 -> 0.0 -0.0 -1.0; child L_Thigh_Link_1 -> L_Thigh_Link; limit lower=-3.14 upper=3.14 effort=500.0 velocity=10.0 -> lower=-0.78 upper=0.78 effort=220.0 velocity=10; origin xyz=0.0 0.048 -0.195 rpy=0 0 0 -> xyz=0.0 0.04 -0.202 rpy=0 0 0; parent L_HipPitch_Link_1 -> L_HipPitch_Link
- joint L_Knee_Joint: child L_Knee_Link_1 -> L_Knee_Link; limit lower=-3.14 upper=3.14 effort=500.0 velocity=10.0 -> lower=0 upper=2.56 effort=95 velocity=10; origin xyz=-0.042753 0.0195 -0.205462 rpy=0 0 0 -> xyz=-0.042753 -0.0195 -0.198462 rpy=0 0 0; parent L_Thigh_Link_1 -> L_Thigh_Link
- joint R_AnklePitch_Joint: child R_AnkleRoll_Link_1 -> R_AnkleRoll_Link; limit lower=-3.14 upper=3.14 effort=500.0 velocity=10.0 -> lower=-0.7 upper=1.05 effort=95 velocity=10; parent R_Knee_Link_1 -> R_Knee_Link
- joint R_AnkleRoll_Joint: child R_Foot_Link_1 -> R_Foot_Link; limit lower=-3.14 upper=3.14 effort=500.0 velocity=10.0 -> lower=-0.42 upper=0.42 effort=95 velocity=10; parent R_AnkleRoll_Link_1 -> R_AnkleRoll_Link
- joint R_HipPitch_Joint: axis 0.0 1.0 -0.0 -> -0.0 1.0 -0.0; child R_HipPitch_Link_1 -> R_HipPitch_Link; limit lower=-3.14 upper=3.14 effort=500.0 velocity=10.0 -> lower=-2.09 upper=1.57 effort=220.0 velocity=10; origin xyz=-0.0075 -0.071 -0.0 rpy=0 0 0 -> xyz=-0.0155 -0.0805 0.0 rpy=0 0 0; parent R_HipRoll_Link_1 -> R_HipRoll_Link
- joint R_HipRoll_Joint: axis -1.0 -0.0 -0.0 -> -1.0 0.0 0.0; child R_HipRoll_Link_1 -> R_HipRoll_Link; limit lower=-3.14 upper=3.14 effort=500.0 velocity=10.0 -> lower=-0.58 upper=0.3 effort=352.0 velocity=10; origin xyz=0.0075 0.0 0.0 rpy=0 0 0 -> xyz=0.0155 0.0 0.0 rpy=0 0 0
- joint R_HipYaw_Joint: child R_Thigh_Link_1 -> R_Thigh_Link; limit lower=-3.14 upper=3.14 effort=500.0 velocity=10.0 -> lower=-0.78 upper=0.78 effort=220.0 velocity=10; origin xyz=0.0 -0.048 -0.195 rpy=0 0 0 -> xyz=0.0 -0.04 -0.202 rpy=0 0 0; parent R_HipPitch_Link_1 -> R_HipPitch_Link
- joint R_Knee_Joint: axis -0.0 -1.0 0.0 -> 0.0 -1.0 0.0; child R_Knee_Link_1 -> R_Knee_Link; limit lower=-3.14 upper=3.14 effort=500.0 velocity=10.0 -> lower=-2.56 upper=0 effort=95 velocity=10; origin xyz=-0.042753 0.0195 -0.205462 rpy=0 0 0 -> xyz=-0.042753 0.0195 -0.198462 rpy=0 0 0; parent R_Thigh_Link_1 -> R_Thigh_Link
- joint WaistYaw_Joint: child WaistYaw_Link_1 -> WaistYaw_Link; limit lower=-3.14 upper=3.14 effort=500.0 velocity=10.0 -> lower=-1.57 upper=1.57 effort=152.0 velocity=10
